Commit message: feat: Migrate firo_calibration and firo_description

File: firo_description/robots/firo.urdf.xacro (robot description, xacro)
@@ -20,5 +20,5 @@
   <xacro:include filename="$(find firo_description)/urdf/wheel.urdf.xacro" />
   <xacro:include filename="$(find firo_description)/urdf/oak-d-w/oak-d-w.urdf.xacro" />
- <!-- Macro to simplify joint definition -->
+  <!-- Macro to simplify joint definition -->
   <xacro:macro name="joint" params="type:='fixed' parent:='base_link' child:='' xyz:='0 0 0' rpy:='0 0 0' axis:='0 0 1' limit_effort:='0.0' limit_velocity:='0.0'">
     <joint name="${child}_joint" type="${type}">
@@ -45,50 +45,66 @@
   <xacro:joint child="back_left_wheel" xyz="${-mechanical.wheel_base/2} ${mechanical.wheel_track/2} ${mechanical.wheel_radius}" type="continuous" axis="0 1 0" limit_effort="7.5" limit_velocity="7.5"/>
   <xacro:joint parent="torso" child="front_camera" xyz="0.3001 0 0.12845"/>
-  <transmission name="front_right_wheel_transmission">
-    <type>transmission_interface/SimpleTransmission</type>
-    <actuator name="front_right_wheel_motor">
-      <mechanicalReduction>1</mechanicalReduction>
-    </actuator>
+  <ros2_control name="GazeboSimSystem" type="system">
+    <hardware>
+      <plugin>libgazebo_ros_control.so</plugin>
+    </hardware>
     <joint name="front_right_wheel_joint">
-    <hardwareInterface>hardware_interface/VelocityJointInterface</hardwareInterface>
+      <command_interface name="velocity">
+        <param name="min">-7.5</param>
+        <param name="max">7.5</param>
+      </command_interface>
+      <state_interface name="position">
+        <param name="initial_value">0.0</param>
+      </state_interface>
+      <state_interface name="velocity" />
+      <state_interface name="effort"/>
     </joint>
-  </transmission>
-  <transmission name="front_left_wheel_transmission">
-    <type>transmission_interface/SimpleTransmission</type>
-    <actuator name="front_left_wheel_motor">
-      <mechanicalReduction>1</mechanicalReduction>
-    </actuator>
     <joint name="front_left_wheel_joint">
-    <hardwareInterface>hardware_interface/VelocityJointInterface</hardwareInterface>
+      <command_interface name="velocity">
+        <param name="min">-7.5</param>
+        <param name="max">7.5</param>
+      </command_interface>
+      <state_interface name="position">
+        <param name="initial_value">0.0</param>
+      </state_interface>
+      <state_interface name="velocity" />
+      <state_interface name="effort"/>
     </joint>
-  </transmission>
-  <transmission name="back_right_wheel_transmission">
-    <type>transmission_interface/SimpleTransmission</type>
-    <actuator name="back_right_wheel_motor">
-      <mechanicalReduction>1</mechanicalReduction>
-    </actuator>
     <joint name="back_right_wheel_joint">
-    <hardwareInterface>hardware_interface/VelocityJointInterface</hardwareInterface>
+      <command_interface name="velocity">
+        <param name="min">-7.5</param>
+        <param name="max">7.5</param>
+      </command_interface>
+      <state_interface name="position">
+        <param name="initial_value">0.0</param>
+      </state_interface>
+      <state_interface name="velocity" />
+      <state_interface name="effort"/>
     </joint>
-  </transmission>
-  <transmission name="back_left_wheel_transmission">
-    <type>transmission_interface/SimpleTransmission</type>
-    <actuator name="back_left_wheel_motor">
-      <mechanicalReduction>1</mechanicalReduction>
-    </actuator>
     <joint name="back_left_wheel_joint">
-    <hardwareInterface>hardware_interface/VelocityJointInterface</hardwareInterface>
+      <command_interface name="velocity">
+        <param name="min">-7.5</param>
+        <param name="max">7.5</param>
+      </command_interface>
+      <state_interface name="position">
+        <param name="initial_value">0.0</param>
+      </state_interface>
+      <state_interface name="velocity" />
+      <state_interface name="effort"/>
     </joint>
-  </transmission>
+  </ros2_control>
   <gazebo>
-    <plugin name="gazebo_ros_control" filename="libgazebo_ros_control.so">
-      <robotNamespace>/</robotNamespace>
-    </plugin>
+    <gazebo>
+      <plugin filename="libgz_ros2_control-system.so" name="gz_ros2_control::GazeboSimROS2ControlPlugin">
+        <hold_joints>true</hold_joints>
+      </plugin>
+    </gazebo>
     <plugin name="p3d_plugin" filename="libgazebo_ros_p3d.so">
-      <alwaysOn>true</alwaysOn>
-      <updateRate>100.0</updateRate>
-      <bodyName>base_link</bodyName>
-      <topicName>ground_truth</topicName>
-      <frameName>map</frameName>
+      <ros>
+        <remapping>odom:=ground_truth</remapping>
+      </ros>
+      <update_rate>100.0</update_rate>
+      <body_name>base_link</body_name>
+      <frame_name>map</frame_name>
     </plugin>
   </gazebo>
