Commit message: feat: odrive can hardware interface urdf

File: firo_description/robots/firo.urdf.xacro (robot description, xacro)
@@ -45,5 +45,5 @@
   <xacro:joint child="back_left_wheel" xyz="${-mechanical.wheel_base/2} ${mechanical.wheel_track/2} ${mechanical.wheel_radius}" type="continuous" axis="0 1 0" limit_effort="7.5" limit_velocity="7.5"/>
   <xacro:joint parent="torso" child="front_camera" xyz="0.3001 0 0.12845"/>
-  <ros2_control name="GazeboSimSystem" type="system">
+  <!-- <ros2_control name="GazeboSimSystem" type="system">
     <hardware>
       <plugin>gz_ros2_control/GazeboSimSystem</plugin>
@@ -93,4 +93,24 @@
       <state_interface name="effort"/>
     </joint>
+  </ros2_control> -->
+  <ros2_control name="odrive_can_left" type="actuator">
+    <hardware>
+      <plugin>odrive_can_driver/OdriveHardwareInterface</plugin>
+      <param name="interface">can0</param>
+    </hardware>
+    <joint name="front_left_wheel_joint">
+      <param name="node_id">10</param>
+      <command_interface name="velocity" />
+      <state_interface name="position" />
+      <state_interface name="velocity" />
+      <state_interface name="effort"/>
+    </joint>
+    <joint name="back_left_wheel_joint">
+      <param name="node_id">11</param>
+      <command_interface name="velocity" />
+      <state_interface name="position" />
+      <state_interface name="velocity" />
+      <state_interface name="effort"/>
+    </joint>
   </ros2_control>
   <gazebo>

Commit message: feat: add right wheels hardware configuration

File: firo_description/robots/firo.urdf.xacro (robot description, xacro)
@@ -94,10 +94,10 @@
     </joint>
   </ros2_control> -->
-  <ros2_control name="odrive_can_left" type="actuator">
+  <ros2_control name="odrive_can_right" type="actuator">
     <hardware>
       <plugin>odrive_can_driver/OdriveHardwareInterface</plugin>
       <param name="interface">can0</param>
     </hardware>
-    <joint name="front_left_wheel_joint">
+    <joint name="front_right_wheel_joint">
       <param name="node_id">10</param>
       <command_interface name="velocity" />
@@ -106,6 +106,26 @@
       <state_interface name="effort"/>
     </joint>
+    <joint name="back_right_wheel_joint">
+      <param name="node_id">11</param>
+      <command_interface name="velocity" />
+      <state_interface name="position" />
+      <state_interface name="velocity" />
+      <state_interface name="effort"/>
+    </joint>
+  </ros2_control>
+  <ros2_control name="odrive_can_left" type="actuator">
+    <hardware>
+      <plugin>odrive_can_driver/OdriveHardwareInterface</plugin>
+      <param name="interface">can0</param>
+    </hardware>
     <joint name="back_left_wheel_joint">
-      <param name="node_id">11</param>
+      <param name="node_id">12</param>
+      <command_interface name="velocity" />
+      <state_interface name="position" />
+      <state_interface name="velocity" />
+      <state_interface name="effort"/>
+    </joint>
+    <joint name="front_left_wheel_joint">
+      <param name="node_id">13</param>
       <command_interface name="velocity" />
       <state_interface name="position" />

Commit message: feat: added lidar,imu,footprint to robot description

File: firo_description/robots/firo.urdf.xacro (robot description, xacro)
@@ -46,4 +46,10 @@
   <xacro:joint child="back_left_wheel" xyz="${-mechanical.wheel_base/2} ${mechanical.wheel_track/2} ${mechanical.wheel_radius}" type="continuous" axis="0 1 0" limit_effort="7.5" limit_velocity="7.5"/>
   <xacro:joint parent="torso" child="front_camera" xyz="0.3001 0 0.12845"/>
+  <link name="lidar_link"/>
+  <xacro:joint parent="torso" child="lidar_link" xyz="0.265 0 0.055" rpy="0 0 0"/>
+  <link name="imu_link"/>
+  <xacro:joint parent="torso" child="imu_link" xyz="0 0 0.023" rpy="0 0 0"/>
+  <link name="base_footprint"/>
+  <xacro:joint parent="base_link" child="base_footprint" xyz="0 0 -0.09" rpy="0 0 0"/>
   <xacro:if value="$(arg gazebo)">
     <ros2_control name="GazeboSimSystem" type="system">

Commit message: fear: added vertical lidar filters, works as should, trying to launch them all at once

File: firo_description/robots/firo.urdf.xacro (robot description, xacro)
@@ -46,6 +46,10 @@
   <xacro:joint child="back_left_wheel" xyz="${-mechanical.wheel_base/2} ${mechanical.wheel_track/2} ${mechanical.wheel_radius}" type="continuous" axis="0 1 0" limit_effort="7.5" limit_velocity="7.5"/>
   <xacro:joint parent="torso" child="front_camera" xyz="0.3001 0 0.12845"/>
-  <link name="lidar_link"/>
-  <xacro:joint parent="torso" child="lidar_link" xyz="0.265 0 0.055" rpy="0 0 0"/>
+  <link name="lidar_horizontal_link"/>
+  <xacro:joint parent="torso" child="lidar_horizontal_link" xyz="0.265 0 0.055" rpy="0 0 0"/>
+  <link name="lidar_vertical_left_link"/>
+  <xacro:joint parent="torso" child="lidar_vertical_left_link" xyz="-0.135 0.2 0.05" rpy="-1.5708 0 0"/>
+  <link name="lidar_vertical_right_link"/>
+  <xacro:joint parent="torso" child="lidar_vertical_right_link" xyz="-0.135 -0.2 0.05" rpy="1.5708 0 0"/>
   <link name="imu_link"/>
   <xacro:joint parent="torso" child="imu_link" xyz="0.025 0 0.023" rpy="0 0 3.14159"/>
